File: corinda.kicad_pcb (KiCad board)
At the start: 2 copper layers, 27 x 35.4 mm, 15 parts, among them J1 Pixels, J2 USB_B_Micro, J3 ExtPwr, J4 ExtPwr2, SW1 RESET, U1 ME6211, U2 ESP-C3-13U, U3 D1_Mini_16p

Commit message: Corinda 1v1
Parts:
- removed the C3 at (125.5, 93.5)
- removed the J4 at (138.9, 97.5)
- added C1: 10uF, Capacitor_SMD:C_0402_1005Metric, F.Cu at (125.8, 98.4)
- added D2: B5819, Diode_SMD:D_SOD-123, F.Cu at (127.4, 94.6)
- added D3: IO4, LED_SMD:LED_0402_1005Metric, F.Cu at (119.5, 68.0)
- added G***: LOGO, LOGO, F.Cu at (121.8, 69.0)
- added J1: USB_B_Micro, Accelerando:USB_Micro_SMD, F.Cu at (131.0, 101.4)
- added P1: RGB=IO9, Accelerando:LED_WS2812B_PLCC2_0x1_8mm_P1.27mm, F.Cu at (139.2, 68.5)
- added P2: RGB, Accelerando:LED_WS2812B_PLCC2_0x1_8mm_P1.27mm, F.Cu at (139.2, 71.2)
- added Q1: SI2307, Package_TO_SOT_SMD:SOT-23, F.Cu at (122.8, 95.8)
- added R1: 2k, Resistor_SMD:R_0402_1005Metric, F.Cu at (119.8, 97.0)
- added R3: 3k3, Resistor_SMD:R_0402_1005Metric, F.Cu at (135.0, 95.0)
- added R4: 3k3, Resistor_SMD:R_0402_1005Metric, F.Cu at (135.0, 96.2)
- added R6: 1k, Resistor_SMD:R_0402_1005Metric, F.Cu at (123.5, 68.0)
- added U1: TP4054, Package_TO_SOT_SMD:SOT-23-5, F.Cu at (120.4, 99.6)
- C2: footprint Capacitor_SMD:C_0805_2012Metric_Pad1.18x1.45mm_HandSolder -> Capacitor_SMD:C_0402_1005Metric
- C3: renamed from C1; value 100nF -> 0u1; footprint Capacitor_SMD:C_0603_1608Metric_Pad1.08x0.95mm_HandSolder -> Capacitor_SMD:C_0402_1005Metric
- C4: value 100nF -> 0u1; footprint Capacitor_SMD:C_0603_1608Metric_Pad1.08x0.95mm_HandSolder -> Capacitor_SMD:C_0402_1005Metric
- D1: value WS2812B_2020 -> CHG; footprint Accelerando:LED_WS2812B_PLCC2_0x1_8mm_P1.27mm -> LED_SMD:LED_0402_1005Metric
- J2: value USB_B_Micro -> BATT; footprint Accelerando:USB_Micro_SMD -> Connector_JST:JST_GH_SM02B-GHS-TB_1x02-1MP_P1.25mm_Horizontal; moved to B.Cu
- J3: value ExtPwr -> QWIIC; footprint Connector_JST:JST_GH_SM02B-GHS-TB_1x02-1MP_P1.25mm_Horizontal -> Connector_JST:JST_SH_SM04B-SRSS-TB_1x04-1MP_P1.00mm_Horizontal
- J4: renamed from J1; value Pixels -> EGON; footprint Connector_JST:JST_XH_S3B-XH-A_1x03_P2.50mm_Horizontal -> Connector_JST:JST_GH_SM03B-GHS-TB_1x03-1MP_P1.25mm_Horizontal
- R2: value 10k -> 2k; footprint Resistor_SMD:R_0603_1608Metric_Pad0.98x0.95mm_HandSolder -> Resistor_SMD:R_0402_1005Metric
- R5: renamed from R1; footprint Resistor_SMD:R_0603_1608Metric_Pad0.98x0.95mm_HandSolder -> Resistor_SMD:R_0402_1005Metric
- SW1: value RESET -> PWR; footprint Accelerando:TVBM02 -> Button_Switch_SMD:SW_SPDT_PCM12; moved to B.Cu
- moved D1 34.2 mm to (119.8, 96.0), turned to 0 degrees
- moved C3 12.6 mm to (126.0, 96.4), turned to 180 degrees
- moved C4 12.5 mm to (135.0, 93.8), turned to 180 degrees
- moved J2 10.1 mm to (139.0, 98.0), turned to 90 degrees
- moved C2 8.79 mm to (119.8, 95.0), turned to 180 degrees
- moved R5 8.00 mm to (128.8, 96.4), turned to 0 degrees
- moved R2 4.92 mm to (123.6, 98.4), turned to 0 degrees
- moved J4 3.55 mm to (132.0, 69.5)
- moved SW1 3.11 mm to (122.0, 99.5), turned to 180 degrees
- moved U3 2.57 mm to (130.2, 83.3)
- moved U2 1.60 mm to (132.0, 95.0), turned to 0 degrees
- moved J3 0.97 mm to (139.2, 97.7), turned to 90 degrees
- renumbered U3 to M1, U1 to U2, U2 to U3
Connections:
- C2 pad 1: /3v3 -> +BATT
- C4 pad 2: /RST -> +3V3
- D1 pad 1: /PIXELS -> /~{CHRG}
- D1 pad 2: GND -> /CHGLED
- J2 pad 1: +5V -> /B+
- J2 pad 2: /IO18/D- -> GND
- J3 pad 1: +5V -> GND
- J3 pad 2: GND -> +3V3
- J3 pad MP: GND -> (no net)
- J4 pad 1: /3v3 -> +3V3
- J4 pad 2: /PIXELS -> /EGON
- M1 pad 8: /3v3 -> +3V3
- R2 pad 1: /3v3 -> /PROG
- R2 pad 2: /RST -> GND
- SW1 pad : (no net) -> GND
- SW1 pad 1: GND -> /B+
- SW1 pad 2: /RST -> +BATT
- U2 pad 5: /3v3 -> +3V3
- U3 pad 1: /3v3 -> +3V3
Routing:
- net +3V3: track 0.00 -> 76.9 mm, vias 0 -> 4
- net /3v3: track 53.0 -> 0.00 mm, vias 2 -> 0
- net /VBUS: track 0.00 -> 24.1 mm
- net /IO1: track 22.7 -> 46.8 mm, vias 0 -> 1
- net /IO4/MTMS: track 16.7 -> 39.0 mm, vias 0 -> 1
- net /PIXELS: track 18.6 -> 0.00 mm, vias 1 -> 0
- net /IO2: track 23.7 -> 42.0 mm, vias 2 -> 1
- net /B+: track 0.00 -> 17.8 mm
- net +5V: track 31.2 -> 19.4 mm, vias 0 -> 2
- net /RST: track 31.7 -> 21.8 mm, vias 5 -> 2
- net +BATT: track 0.00 -> 9.55 mm, vias 0 -> 2
- net /EGON: track 0.00 -> 7.69 mm
- net GND: track 21.9 -> 29.4 mm, vias 0 -> 14
- net Net-(P1-Pad1): track 0.00 -> 7.15 mm
- net /IO10: track 27.1 -> 22.0 mm
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- removed copper zone on F.Cu, net GND
Other:
- board text added: "1v2 ©2023 accelerando.io"
- board text added: "3v RST IO4 IO5 I6 I7 IO8 IO9"
- board text added: "Accelerando {dblquote}Corinda{dblquote}"
- board text added: "G 3 D C"
- board text added: "GND"
- board text added: "IO0 IO1 IO2 IO3 D+ D- Tx Rx IO10"
- board text added: "IO10 IO0"
- board text added: "SCL SDA"
- board text added: "SCLK MISO MOSI ~{SS}"
- board text added: "SDA SCL IO20 IO21"
- board text added: "{dblquote}Corinda{dblquote} 1v2"
- board text removed: "- +"
- board text removed: "Accelerando {dblquote}Corinda{dblquote} 1v0"
- board text removed: "D9"
- board text removed: "©2022 accelerando.com.au"
